File: pcb/splitflap_speaker_board/splitflap_speaker_board.kicad_pcb (KiCad board)
At the start: 4 copper layers, 130 x 75 mm, 81 parts, among them J14 L_out, J15 R_out, J8 POT, Q1 BSS138, Q2 BSS138, U1 TPS562243DRLR, U2 LM1084-5.0, U3 PCM5122PW, U4 MAX9744

Commit message: Another DRC test, changed company name
Other:
- board text added: "Splitflap Speaker Board Design: Axi Eltanin Engineering Co. Rev 1.2"
- board text removed: "Splitflap Speaker Board Design: Axi Eltanin Industrial Co. Rev 1.2"
