File: pcb/splitflap_speaker_board/splitflap_speaker_board.kicad_pcb (KiCad board)
At the start: 4 copper layers, 130 x 75 mm, 81 parts, among them J14 L_out, J15 R_out, J8 POT, Q1 BSS138, Q2 BSS138, U1 TPS562243DRLR, U2 LM1084-5.0, U3 PCM5122PW, U4 MAX9744

Commit message: Audio layout fixes: pot filter, 12 V feed, AVDD ferrite, antenna keepout
- Pot line moved to the bottom layer away from the speaker terminals, with
  an RC filter (R16 1k, C38 100nF) before the shielded run to the amp's VOL
- 12 V feed no longer runs around the DAC: it drops down east of the DAC
  to C36 and crosses under the amp on the bottom layer to the left PVDD side
- DAC AVDD fed through its own ferrite (FB2) from the 3.3 V trunk instead of
  the amp's VDD branch
- DAC ATT0/MAST grounded at the chip; their long strap traces removed
- Copper-pour keepout under the Pi Zero 2 W antenna edge (all layers)

Zone fills were not regenerated: refill zones in KiCad before DRC/plots.

Co-Authored-By: Claude Opus 5.5 <noreply@anthropic.com>
Claude-Session: https://claude.ai/code/session_01FgEhnNNRCVfH3GgykTypvy
Parts:
- added C38: 0.1uF_0603_16V, Capacitor_SMD:C_0603_1608Metric, F.Cu at (148.4, 142.6)
- added FB2: 220ohm MPZ2012S221A TDK, Inductor_SMD:L_0805_2012Metric, F.Cu at (145.6, 123.6)
- added R16: 1k, Resistor_SMD:R_0603_1608Metric, F.Cu at (150.8, 141.0)
Connections:
- C12 pad 2: +3.3V -> /AVDD
- C14 pad 1: +3.3V -> /AVDD
- U3 pad 8: +3.3V -> /AVDD
- U4 pad 8: /POT_IN -> /VOL
Routing:
- net GND: track 274.9 -> 141.7 mm, vias 48 -> 44
- net /AVDD: track 0.00 -> 20.8 mm, vias 0 -> 2
- net /VOL: track 0.00 -> 20.8 mm, vias 0 -> 2
- net +12V: track 189.7 -> 170.5 mm, vias 2 -> 4
- net /POT_IN: track 56.9 -> 45.2 mm, vias 2 -> 1
- net +3.3V: track 337.9 -> 326.6 mm, vias 5 -> 6
