File: pcb/splitflap_speaker_board/splitflap_speaker_board.kicad_sch (KiCad schematic)
At the start: 78 parts, among them J13 12V in, J14 L_out, J15 R_out, J2 Splitflap_out, J3 SNOOZE, J4 LED, J6 RPI, J7 Illu header, J8 POT, Q1 BSS138, Q2 BSS138, U1 TPS562243DRLR, U2 LM1084-5.0, U3 PCM5122PW, U4 MAX9744

Commit message: Fix speaker board blockers and match software to the board pins
Board + schematic (kept in sync; netlists now match pad for pad):
- Buck feedback R7 100k -> 10k so the "+7V" rail is 6.6 V, not 1.2 V
- PCM5122: AVDD tied to +3.3V; SCK grounded; MODE2 grounded for
  hardware mode with ATT1/ATT2/AGNS grounded (0 dB, 2 Vrms)
- MAX9744 analog volume mode: slide pot wiper on SDA/VOL, SCLK to GND
  (filterless); amp taken off the I2C bus
- MAX9744 exposed pad + thermal vias on GND (EP pin added to symbol)
- Left channel input/feedback resistors moved to the correct pins
- LED strip data moved from GPIO5 to GPIO10 (SPI0 MOSI)
- C15/C16 (2.2 uF straight on the DAC outputs) marked DNP
- Schematic: connector refs, Pi socket and L1/C4/C28 footprints and
  J14 pin order updated to match the board; speaker +/- silk moved
  next to the terminals

Software:
- Replace I2C amp driver and ADS1115 pot reader with GPIO control of
  DAC XSMT/ATT0/MAST/FLT and amp SHDN/MUTE
- Web volume slider now sets MPD stream volume
- Buttons on GPIO0 (snooze) and GPIO12 (LED); docs updated for the
  Pi Zero W and the hifiberry-dac overlay

Zone fills were not regenerated: refill zones in KiCad before DRC/plots.

Co-Authored-By: Claude Opus 5.5 <noreply@anthropic.com>
Claude-Session: https://claude.ai/code/session_01FgEhnNNRCVfH3GgykTypvy
Parts:
- C15, C16: now not fitted
- C28: footprint Capacitor_SMD:C_0201_0603Metric -> Capacitor_SMD:C_0402_1005Metric
- C4: footprint Capacitor_SMD:C_0603_1608Metric -> Capacitor_SMD:C_0805_2012Metric
- L1: footprint Inductor_SMD:L_0603_1608Metric -> Inductor_SMD:L_Bourns_SRN6045TA
- R7: value 100k_0603 -> 10k; Display 30k -> 10k; JLCPCB ID C25803 -> C25804; LCSC C25803 -> C25804; Part Number RC0603FR-07100KL -> RC0603FR-0710KL; Specifications 100K, 1%, 1/10W, 0603 -> 10K, 1%, 1/10W, 0603
- Raspberry: renamed from J6; footprint Connector_PinHeader_2.54mm:PinHeader_2x20_P2.54mm_Vertical -> Connector_PinSocket_2.54mm:PinSocket_2x20_P2.54mm_Vertical
- renumbered J13 to 12V, J7 to Illu, J4 to LED, J3 to Snooze, J2 to Splitflap
Connections:
- net AVDD is gone; now on net +3.3V: C12.2, C14.1, U3.8 (AVDD)
- net DGND is gone; now on net GND: U3.16 (ADR2/GPIO2/DOUT), U3.20 (SCK), U3.24 (ADR1/MISO/FMT)
- net GP8 is gone; now on net LED: Raspberry.19 (Pin_19)
- net +3.3V: no longer U3.18 (MODE2/MS)
- net FBL: now also R10.1, U4.17 (FBL); no longer R10.2, U4.16 (INL)
- net GND: now also U3.11 (SDA/MOSI/ATT2), U3.12 (SCL/MC/ATT1), U3.15 (GPIO3/AGNS), U3.18 (MODE2/MS), U4.45 (EP), U4.9 (SCLK)
- net INL: now also R10.2, U4.16 (INL); no longer R10.1, U4.17 (FBL)
- net LED: no longer Raspberry.29 (Pin_29)
- net POT_IN: now also U4.8 (SDA/VOL); no longer U3.11 (SDA/MOSI/ATT2)
- net SCL_3.3V: no longer U4.9 (SCLK)
- net SDA_3.3V: no longer U4.8 (SDA/VOL)
- net SPK_L+: now reaches Bead1.2, C32.1
- net SPK_L+: now also J14.2 (Pin_2); no longer J14.1 (Pin_1)
- net SPK_L-: now reaches Bead2.2, C33.2
- net SPK_L-: now also J14.1 (Pin_1); no longer J14.2 (Pin_2)
- no-connect marks 26 -> 25
Other:
- moved on the sheet: R10

Commit message: Mirror Pi socket for a face-up Pi Zero W and re-route the header
The Pi Zero W now mounts component side up with its header pins pointing
down into the board's socket. That mirrors the pinout, so:

- New footprint eltanin_footprints:PinSocket_2x20_P2.54mm_Vertical_PiFaceUp
  (stock 2x20 socket with mirrored pad numbering), pin 1 at the east end
- Re-routed 3.3 V, I2C, I2S (BCK/LRCK/DIN) and SPI MOSI to their new pins;
  5 V and GND reach the Pi through the inner planes as before
- GPIO signals moved to free pins: snooze GPIO27, LED button GPIO4,
  amp ~SHDN GPIO13, amp MUTE GPIO25
- DAC straps tied on the board instead of Pi GPIOs: XSMT high,
  MAST/ATT0/FLT low
- Schematic updated to match; software config and docs follow

Zone fills were not regenerated: refill zones in KiCad before DRC/plots.

Co-Authored-By: Claude Opus 5.5 <noreply@anthropic.com>
Claude-Session: https://claude.ai/code/session_01FgEhnNNRCVfH3GgykTypvy
Parts:
- Raspberry: footprint Connector_PinSocket_2.54mm:PinSocket_2x20_P2.54mm_Vertical -> eltanin_footprints:PinSocket_2x20_P2.54mm_Vertical_PiFaceUp
Connections:
- net +3.3V: now also U3.25 (XSMT)
- net GND: now also Raspberry.6 (Pin_6), U3.13 (GPIO5/ATT0), U3.14 (GPIO4/MAST), U3.19 (GPIO6/FLT)
- net ILLU: now also Raspberry.7 (Pin_7); no longer Raspberry.32 (Pin_32)
- net MUTE: now also Raspberry.22 (Pin_22); no longer Raspberry.18 (Pin_18)
- net SHND: now also Raspberry.33 (Pin_33); no longer Raspberry.7 (Pin_7)
- net SNOOZE: now also Raspberry.13 (Pin_13); no longer Raspberry.27 (Pin_27)
- net GP3: no longer names the net of Raspberry.15 (Pin_15)
- net GP3: no longer U3.25 (XSMT)
- net GP4: no longer names the net of Raspberry.16 (Pin_16)
- net GP4: no longer U3.14 (GPIO4/MAST)
- net GP5: no longer names the net of Raspberry.36 (Pin_36)
- net GP5: no longer U3.13 (GPIO5/ATT0)
- removed net GP6: Raspberry.22 (Pin_22), U3.19 (GPIO6/FLT)
- no-connect marks 25 -> 28

Commit message: Audio layout fixes: pot filter, 12 V feed, AVDD ferrite, antenna keepout
- Pot line moved to the bottom layer away from the speaker terminals, with
  an RC filter (R16 1k, C38 100nF) before the shielded run to the amp's VOL
- 12 V feed no longer runs around the DAC: it drops down east of the DAC
  to C36 and crosses under the amp on the bottom layer to the left PVDD side
- DAC AVDD fed through its own ferrite (FB2) from the 3.3 V trunk instead of
  the amp's VDD branch
- DAC ATT0/MAST grounded at the chip; their long strap traces removed
- Copper-pour keepout under the Pi Zero 2 W antenna edge (all layers)

Zone fills were not regenerated: refill zones in KiCad before DRC/plots.

Co-Authored-By: Claude Opus 5.5 <noreply@anthropic.com>
Claude-Session: https://claude.ai/code/session_01FgEhnNNRCVfH3GgykTypvy
Parts:
- added C38: 0.1uF_0603_16V, Capacitor_SMD:C_0603_1608Metric, symbol PCM_4ms_Capacitor:0.1uF_0603_16V
- added FB2: 220ohm MPZ2012S221A TDK, Inductor_SMD:L_0805_2012Metric, symbol Device:FerriteBead
- added R16: 1k, Resistor_SMD:R_0603_1608Metric, symbol Device:R_Small
Connections:
- net +3.3V: now also FB2.2; no longer C12.2, C14.1, U3.8 (AVDD)
- net GND: now also C38.2
- net POT_IN: now also R16.2; no longer U4.8 (SDA/VOL)
- new net AVDD: C12.2, C14.1, FB2.1, U3.8 (AVDD)
- new net VOL: C38.1, R16.1, U4.8 (SDA/VOL)
